File: LightProcessor/LightProcessor.kicad_sch (KiCad schematic)
At the start: 30 parts, among them IC1 STM32G474RET6, J1 USB_C_Receptacle_USB2.0_16P, SW10 Tactile_6mm, U1 STLINK-V3MODS, U3 AP2112K-3.3, Y1 16MHz

Commit message: Added additional functions
Parts:
- added U2: LM324, symbol Amplifier_Operational:LM324

Commit message: Update PCB design
Parts:
- removed ADC5: Conn_Coaxial, Connector_Coaxial:BNC_TEConnectivity_1478035_Horizontal, symbol Connector:Conn_Coaxial
- added C16: 0.1, Capacitor_SMD:C_0805_2012Metric_Pad1.18x1.45mm_HandSolder, symbol Device:C
- added C22: 0.1u, Capacitor_SMD:C_0805_2012Metric_Pad1.18x1.45mm_HandSolder, symbol Device:C
- added D2, D3, D4, D5: D, Diode_SMD:D_0805_2012Metric, symbol Device:D
- added D22, D30, D31, D32, D33, D35, D36, D37, D38, D40, D41, D42, D43, D45, D46, D47, D48: LED, LED_SMD:LED_0805_2012Metric, symbol Device:LED
- added D23, D29, D34, D39, D44: RED, LED_SMD:LED_0805_2012Metric, symbol Device:LED
- added D49: GREEN, LED_SMD:LED_0805_2012Metric, symbol Device:LED
- added DAC1: Conn_Coaxial, 5415025-2:CONN BNC JACK RA 50 OHM PCB, symbol Connector:Conn_Coaxial
- added FB1: FerriteBead, Capacitor_SMD:C_0805_2012Metric, symbol Device:FerriteBead
- added J2: PJ-202B, PJ_202B:CUI_PJ-202B, symbol PJ-202B:PJ-202B
- added R1, R17, R25, R9: 500K, Resistor_THT:R_Axial_DIN0207_L6.3mm_D2.5mm_P15.24mm_Horizontal, symbol Device:R
- added R10, R12, R18, R2, R20, R26, R28, R4: 330K, Resistor_THT:R_Axial_DIN0207_L6.3mm_D2.5mm_P15.24mm_Horizontal, symbol Device:R
- added R11, R19, R27, R3: 1M, Resistor_THT:R_Axial_DIN0207_L6.3mm_D2.5mm_P15.24mm_Horizontal, symbol Device:R
- added R13, R21, R29, R5: 250K, Resistor_THT:R_Axial_DIN0207_L6.3mm_D2.5mm_P15.24mm_Horizontal, symbol Device:R
- added R14, R22, R30, R6: 110K, Resistor_THT:R_Axial_DIN0207_L6.3mm_D2.5mm_P15.24mm_Horizontal, symbol Device:R
- added R53, R54, R55, R56, R57, R58, R59, R60, R68, R69, R70, R71, R72, R73, R74, R75, R76, R77, R78, R79, R80, R81, R82, R83, R84, R85, R86, R87, R88, R89, R90: 100K, Resistor_SMD:R_0805_2012Metric, symbol Device:R
- added R91: 0, Resistor_SMD:R_0805_2012Metric, symbol Device:R
- added SW11, SW7, SW8, SW9: SW_SP5T_NR01105, Button_Switch_THT:SW_NKK_NR01, symbol Switch:SW_SP5T_NR01105
- added U10, U12, U13: SN74HC4066N, N14, symbol SN74HC4066N:SN74HC4066N
- added U11: SN74HC4066N, SN74HC4066N:N14, symbol SN74HC4066N:SN74HC4066N
- added U4, U6, U7, U8, U9: LM324, LM324N_NOPB:DIP825W47P254L1917H533Q14, symbol Amplifier_Operational:LM324
- ADC1, ADC2, ADC3, ADC4: footprint Connector_Coaxial:BNC_TEConnectivity_1478035_Horizontal -> 5415025-2:CONN BNC JACK RA 50 OHM PCB
- C11: value 1u -> 0.1u
- U2: footprint (none) -> LM324N_NOPB:DIP825W47P254L1917H533Q14
Connections:
- net +3.3V: now also IC1.1 (VBAT), D22.2 (A), FB1.2, R53.2, R55.2, R57.2, R59.2, SW11.C (Common), SW7.C (Common), SW8.C (Common), SW9.C (Common), U10.14 (VCC), U11.14 (VCC), U12.14 (VCC), U13.14 (VCC)
- net +5V: now also U2.4 (V+), J2.1, U4.4 (V+), U6.4 (V+), U7.4 (V+), U8.4 (V+), U9.4 (V+); no longer J1.A4 (VBUS), J1.A9 (VBUS), J1.B4 (VBUS), J1.B9 (VBUS)
- net ADC1_IN3: now also D3.2 (A), U9.6 (-), U9.7; no longer ADC1.1 (In), IC1.14 (PA2)
- net ADC2_IN3: now also D4.2 (A), U9.8, U9.9 (-); no longer ADC2.1 (In), IC1.20 (PA6)
- net ADC3_IN1: now also D5.2 (A), U9.13 (-), U9.14; no longer ADC3.1 (In), IC1.25 (PB1)
- net ADC4_IN5: now also D2.2 (A), U9.1, U9.2 (-); no longer ADC4.1 (In), IC1.37 (PB15)
- net GND: now also J1.S1 (SHIELD), J2.2, J2.3, R68.1, R69.1, R70.1, R71.1, R72.1, R73.1, R74.1, R75.1, R76.1, R77.1, R78.1, R79.1, R80.1, R81.1, R82.1, R83.1, R84.1, R85.1, R86.1, R87.1, R88.1, R89.1, R90.1, R91.1, SW11.MP, SW7.MP, SW8.MP, SW9.MP, U10.7 (GND), U11.7 (GND), U12.7 (GND), U13.7 (GND), U9.11 (V-); no longer ADC1.2 (Ext), ADC2.2 (Ext), ADC3.2 (Ext), ADC4.2 (Ext), IC1.27 (VSSA)
- net ~{RESET}: now also U1.31 (NRST)
- net ADC2_BUFFER: now reaches U2.1
- net ADC2_BUFFER: now also U2.2 (-), R11.1, R13.1, R9.1, U11.11 (4A)
- net ADC2_RAW: now reaches U2.3 (+)
- net ADC2_RAW: now also ADC2.1 (In)
- net ADC3_RAW: now reaches U2.10 (+)
- net ADC3_RAW: now also ADC3.1 (In)
- net ADC3_BUFFER: now reaches U2.8
- net ADC3_BUFFER: now also U2.9 (-), R17.1, R19.1, R21.1, U12.11 (4A)
- net ADC1_MOD1_IND: now reaches IC1.10 (PC2)
- net ADC1_MOD1_IND: now also D40.2 (A), SW9.1, U10.6 (3C)
- net ADC1_MOD2_IND: now reaches IC1.11 (PC3)
- net ADC1_MOD2_IND: now also D42.2 (A), SW9.2, U10.5 (2C)
- net ADC1_MOD3_IND: now reaches IC1.12 (PA0)
- net ADC1_MOD3_IND: now also D43.2 (A), SW9.3, U10.13 (1C)
- net ADC1_MOD4_IND: now reaches IC1.13 (PA1)
- net ADC1_MOD4_IND: now also D41.2 (A), SW9.4, U10.12 (4C)
- net DAC_OUT: now reaches IC1.18 (PA4)
- net DAC_OUT: now also DAC1.1 (In)
- net ADC3_MOD4_IND: now reaches IC1.21 (PA7)
- net ADC3_MOD4_IND: now also D46.2 (A), SW11.4, U12.12 (4C)
- net ADC3_MOD3_IND: now reaches IC1.22 (PC4)
- net ADC3_MOD3_IND: now also D48.2 (A), SW11.3, U12.6 (3C)
- net ADC3_MOD2_IND: now reaches IC1.23 (PC5)
- net ADC3_MOD2_IND: now also D47.2 (A), SW11.2, U12.5 (2C)
- net ADC3_MOD1_IND: now reaches IC1.24 (PB0)
- net ADC3_MOD1_IND: now also D45.2 (A), SW11.1, U12.13 (1C)
- net ADC3_IDLE_IND: now reaches IC1.26 (PB2)
- net ADC3_IDLE_IND: now also D44.2 (A), SW11.5
- net at IC1.29 (VDDA): now also C16.1, C22.1
- net ADC4_MOD4_IND: now reaches IC1.33 (PB11)
- net ADC4_MOD4_IND: now also D31.2 (A), SW7.4, U13.12 (4C)
- net ADC4_MOD3_IND: now reaches IC1.34 (PB12)
- net ADC4_MOD3_IND: now also D33.2 (A), SW7.3, U13.6 (3C)
- net ADC4_MOD2_IND: now reaches IC1.35 (PB13)
- net ADC4_MOD2_IND: now also D32.2 (A), SW7.2, U13.5 (2C)
- net ADC4_MOD1_IND: now reaches IC1.36 (PB14)
- net ADC4_MOD1_IND: now also D30.2 (A), SW7.1, U13.13 (1C)
- net ADC2_MOD4_IND: now reaches IC1.38 (PC6)
- net ADC2_MOD4_IND: now also D36.2 (A), SW8.4, U11.12 (4C)
- net ADC2_MOD3_IND: now reaches IC1.39 (PC7)
- net ADC2_MOD3_IND: now also D38.2 (A), SW8.3, U11.6 (3C)
- net ADC2_MOD2_IND: now reaches IC1.40 (PC8)
- net ADC2_MOD2_IND: now also D37.2 (A), SW8.2, U11.5 (2C)
- net ADC2_MOD1_IND: now reaches IC1.41 (PC9)
- net ADC2_MOD1_IND: now also D35.2 (A), SW8.1, U11.13 (1C)
- net RX_IND: now reaches IC1.43 (PA9)
- net RX_IND: now also D49.2 (A)
- net TX_IND: now reaches IC1.44 (PA10)
- net TX_IND: now also D23.2 (A)
- net D-: now reaches IC1.45 (PA11)
- net D-: now also J1.A7 (D-)
- net D+: now reaches IC1.46 (PA12)
- net D+: now also J1.A6 (D+)
- net ADC4_IDLE_IND: now reaches IC1.8 (PC0)
- net ADC4_IDLE_IND: now also D29.2 (A), SW7.5
- net ADC1_IDLE_IND: now reaches IC1.9 (PC1)
- net ADC1_IDLE_IND: now also D39.2 (A), SW9.5
- net ADC1_RAW: now reaches U2.5 (+)
- net ADC1_RAW: now also ADC1.1 (In)
- net ADC1_BUFFER: now reaches U2.6 (-)
- net ADC1_BUFFER: now also U2.7, R1.1, R3.1, R5.1, U10.11 (4A)
- net ADC4_RAW: now reaches U2.12 (+)
- net ADC4_RAW: now also ADC4.1 (In)
- net ADC4_BUFFER: now reaches U2.13 (-)
- net ADC4_BUFFER: now also U2.14, R25.1, R27.1, R29.1, U13.11 (4A)
- net AGND: now reaches U2.11 (V-)
- net AGND: now also ADC1.2 (Ext), ADC2.2 (Ext), ADC3.2 (Ext), ADC4.2 (Ext), IC1.27 (VSSA), DAC1.2 (Ext), R10.2, R12.2, R14.2, R18.2, R2.2, R20.2, R22.2, R26.2, R28.2, R30.2, R4.2, R6.2, R91.2, U4.11 (V-), U6.11 (V-), U7.11 (V-), U8.11 (V-)
- net ADC5_IN1 renamed ADC2_IDLE_IND
- net ADC2_IDLE_IND: now also D34.2 (A), SW8.5
- net PA15: no longer names the net of IC1.51 (PA15)
- net PB3: no longer names the net of IC1.56 (PB3)
- net PB4: no longer names the net of IC1.57 (PB4)
- net PB5: no longer names the net of IC1.58 (PB5)
- net PB6: no longer names the net of IC1.59 (PB6)
- net PB7: no longer names the net of IC1.60 (PB7)
- net PB8: no longer names the net of IC1.61 (PB8-BOOT0)
- net PB9: no longer names the net of IC1.62 (PB9)
- net PC10: no longer names the net of IC1.52 (PC10)
- net PC11: no longer names the net of IC1.53 (PC11)
- new net: R55.1, R56.2, U9.10 (+)
- new net: D32.1 (K), R71.2
- new net: R25.2, R26.1, U8.5 (+)
- new net: D44.1 (K), R83.2
- new net: R53.1, R54.2, U9.5 (+)
- new net: R57.1, R58.2, U9.12 (+)
- new net: R59.1, R60.2, U9.3 (+)
- new net: D45.1 (K), R84.2
- new net: D33.1 (K), R72.2
- new net: R19.2, R20.1, U7.5 (+)
- new net: R21.2, R22.1, U7.12 (+)
- new net: D40.1 (K), R79.2
- new net: D43.1 (K), R82.2
- new net: R3.2, R4.1, U4.5 (+)
- new net: R5.2, R6.1, U4.10 (+)
- new net: D47.1 (K), R86.2
- new net: D22.1 (K), R88.2
- new net: R1.2, R2.1, U4.3 (+)
- new net: D2.1 (K), IC1.37 (PB15)
- new net: D41.1 (K), R80.2
- new net: D39.1 (K), R78.2
- new net: D38.1 (K), R77.2
- new net: R10.1, R9.2, U6.3 (+)
- new net: D36.1 (K), R75.2
- new net: D34.1 (K), R73.2
- new net: D48.1 (K), R87.2
- new net: D49.1 (K), R90.2
- new net: D3.1 (K), IC1.14 (PA2)
- new net: D4.1 (K), IC1.20 (PA6)
- new net: D5.1 (K), IC1.25 (PB1)
- new net: R11.2, R12.1, U6.5 (+)
- new net: C16.2, C22.2, FB1.1
- new net: R29.2, R30.1, U8.3 (+)
- new net: D30.1 (K), R69.2
- new net: R27.2, R28.1, U8.10 (+)
- new net: D42.1 (K), R81.2
- new net: D23.1 (K), R89.2
- new net: R13.2, R14.1, U6.12 (+)
- new net: D29.1 (K), R68.2
- new net: D37.1 (K), R76.2
- new net: D46.1 (K), R85.2
- new net: R17.2, R18.1, U7.3 (+)
- new net: D31.1 (K), R70.2
- new net: D35.1 (K), R74.2
- new net: J1.A4 (VBUS), J1.A9 (VBUS), J1.B4 (VBUS), J1.B9 (VBUS)
- new net ADC1_MOD1: U10.8 (3A), U4.1, U4.2 (-)
- new net ADC1_MOD2: U10.4 (2A), U4.6 (-), U4.7
- new net ADC1_MOD3: U10.1 (1A), U4.8, U4.9 (-)
- new net ADC1_SCALE: R54.1, U10.10 (4B), U10.2 (1B), U10.3 (2B), U10.9 (3B)
- new net ADC2_MOD1: U11.1 (1A), U6.1, U6.2 (-)
- new net ADC2_MOD2: U11.4 (2A), U6.6 (-), U6.7
- new net ADC2_MOD3: U11.8 (3A), U6.13 (-), U6.14
- new net ADC2_SCALE: R56.1, U11.10 (4B), U11.2 (1B), U11.3 (2B), U11.9 (3B)
- new net ADC3_MOD1: U12.1 (1A), U7.1, U7.2 (-)
- new net ADC3_MOD2: U12.4 (2A), U7.6 (-), U7.7
- new net ADC3_MOD3: U12.8 (3A), U7.13 (-), U7.14
- new net ADC3_SCALE: R58.1, U12.10 (4B), U12.2 (1B), U12.3 (2B), U12.9 (3B)
- new net ADC4_MOD1: U13.1 (1A), U8.6 (-), U8.7
- new net ADC4_MOD2: U13.4 (2A), U8.8, U8.9 (-)
- new net ADC4_MOD3: U13.8 (3A), U8.1, U8.2 (-)
- new net ADC4_SCALE: R60.1, U13.10 (4B), U13.2 (1B), U13.3 (2B), U13.9 (3B)
- no-connect marks 30 -> 7
Other:
- note added: "ADC Buffer"
- note added: "ADC1 MODS"
- note added: "ADC2 MODS"
- note added: "ADC3 MODS"
- note added: "ADC4 MODS"
- note added: "COM LED Indicator"
- note added: "Power LED Indicator"
- moved on the sheet: ADC1, ADC2, ADC3, ADC4, C11, C15, C18, C19, C21, C5, C6, H1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
